Commit message: Second commit: Lan thu hai mong la thanh cong

File: robot_2_description/urdf/robot_2.xacro (robot description, xacro)
@@ -7,10 +7,10 @@
 <link name="base_link">
   <inertial>
-    <origin xyz="0.030778695710215853 0.00017187958403205029 0.0780034263273014" rpy="0 0 0"/>
+    <origin xyz="-0.030778695710215853 -0.00017187958403205029 0.0780034263273014" rpy="0 0 0"/>
     <mass value="6.148868144226647"/>
-    <inertia ixx="0.012471" iyy="0.038142" izz="0.040818" ixy="-6.8e-05" iyz="-2e-05" ixz="-0.007561"/>
+    <inertia ixx="0.012471" iyy="0.038142" izz="0.040818" ixy="-6.8e-05" iyz="-2e-05" ixz="0.007561"/>
   </inertial>
   <visual>
-    <origin xyz="0 0 0" rpy="0 0 0"/>
+    <origin xyz="0 0 0" rpy="0 0 3.141592653589793"/>
     <geometry>
       <mesh filename="file://$(find robot_2_description)/meshes/base_link.stl" scale="0.001 0.001 0.001"/>
@@ -19,5 +19,5 @@
   </visual>
   <collision>
-    <origin xyz="0 0 0" rpy="0 0 0"/>
+    <origin xyz="0 0 0" rpy="0 0 3.141592653589793"/>
     <geometry>
       <mesh filename="file://$(find robot_2_description)/meshes/base_link.stl" scale="0.001 0.001 0.001"/>
@@ -32,5 +32,5 @@
   </inertial>
   <visual>
-    <origin xyz="0.10312 -0.0505 -0.0351" rpy="0 0 0"/>
+    <origin xyz="-0.10312 0.0505 -0.0351" rpy="0 0 3.141592653589793"/>
     <geometry>
       <mesh filename="file://$(find robot_2_description)/meshes/right_steering_1.stl" scale="0.001 0.001 0.001"/>
@@ -39,5 +39,5 @@
   </visual>
   <collision>
-    <origin xyz="0.10312 -0.0505 -0.0351" rpy="0 0 0"/>
+    <origin xyz="-0.10312 0.0505 -0.0351" rpy="0 0 3.141592653589793"/>
     <geometry>
       <mesh filename="file://$(find robot_2_description)/meshes/right_steering_1.stl" scale="0.001 0.001 0.001"/>
@@ -52,5 +52,5 @@
   </inertial>
   <visual>
-    <origin xyz="0.10312 0.0505 -0.0351" rpy="0 0 0"/>
+    <origin xyz="-0.10312 -0.0505 -0.0351" rpy="0 0 3.141592653589793"/>
     <geometry>
       <mesh filename="file://$(find robot_2_description)/meshes/left_steering_1.stl" scale="0.001 0.001 0.001"/>
@@ -59,5 +59,5 @@
   </visual>
   <collision>
-    <origin xyz="0.10312 0.0505 -0.0351" rpy="0 0 0"/>
+    <origin xyz="-0.10312 -0.0505 -0.0351" rpy="0 0 3.141592653589793"/>
     <geometry>
       <mesh filename="file://$(find robot_2_description)/meshes/left_steering_1.stl" scale="0.001 0.001 0.001"/>
@@ -72,5 +72,5 @@
   </inertial>
   <visual>
-    <origin xyz="-0.097623 0.083 -0.0351" rpy="0 0 0"/>
+    <origin xyz="0.097623 -0.083 -0.0351" rpy="0 0 3.141592653589793"/>
     <geometry>
       <mesh filename="file://$(find robot_2_description)/meshes/left_rear_wheel_1.stl" scale="0.001 0.001 0.001"/>
@@ -79,5 +79,5 @@
   </visual>
   <collision>
-    <origin xyz="-0.097623 0.083 -0.0351" rpy="0 0 0"/>
+    <origin xyz="0.097623 -0.083 -0.0351" rpy="0 0 3.141592653589793"/>
     <geometry>
       <mesh filename="file://$(find robot_2_description)/meshes/left_rear_wheel_1.stl" scale="0.001 0.001 0.001"/>
@@ -92,5 +92,5 @@
   </inertial>
   <visual>
-    <origin xyz="-0.098035 -0.083 -0.0351" rpy="0 0 0"/>
+    <origin xyz="0.098035 0.083 -0.0351" rpy="0 0 3.141592653589793"/>
     <geometry>
       <mesh filename="file://$(find robot_2_description)/meshes/right_rear_wheel_1.stl" scale="0.001 0.001 0.001"/>
@@ -99,5 +99,5 @@
   </visual>
   <collision>
-    <origin xyz="-0.098035 -0.083 -0.0351" rpy="0 0 0"/>
+    <origin xyz="0.098035 0.083 -0.0351" rpy="0 0 3.141592653589793"/>
     <geometry>
       <mesh filename="file://$(find robot_2_description)/meshes/right_rear_wheel_1.stl" scale="0.001 0.001 0.001"/>
@@ -112,5 +112,5 @@
   </inertial>
   <visual>
-    <origin xyz="0.10005 -0.082822 -0.0351" rpy="0 0 0"/>
+    <origin xyz="-0.10005 0.082822 -0.0351" rpy="0 0 3.141592653589793"/>
     <geometry>
       <mesh filename="file://$(find robot_2_description)/meshes/right_front_wheel_1.stl" scale="0.001 0.001 0.001"/>
@@ -119,5 +119,5 @@
   </visual>
   <collision>
-    <origin xyz="0.10005 -0.082822 -0.0351" rpy="0 0 0"/>
+    <origin xyz="-0.10005 0.082822 -0.0351" rpy="0 0 3.141592653589793"/>
     <geometry>
       <mesh filename="file://$(find robot_2_description)/meshes/right_front_wheel_1.stl" scale="0.001 0.001 0.001"/>
@@ -132,5 +132,5 @@
   </inertial>
   <visual>
-    <origin xyz="0.10005 0.082822 -0.0351" rpy="0 0 0"/>
+    <origin xyz="-0.10005 -0.082822 -0.0351" rpy="0 0 3.141592653589793"/>
     <geometry>
       <mesh filename="file://$(find robot_2_description)/meshes/left_front_wheel_1.stl" scale="0.001 0.001 0.001"/>
@@ -139,5 +139,5 @@
   </visual>
   <collision>
-    <origin xyz="0.10005 0.082822 -0.0351" rpy="0 0 0"/>
+    <origin xyz="-0.10005 -0.082822 -0.0351" rpy="0 0 3.141592653589793"/>
     <geometry>
       <mesh filename="file://$(find robot_2_description)/meshes/left_front_wheel_1.stl" scale="0.001 0.001 0.001"/>
@@ -146,5 +146,5 @@
 </link>
 <joint name="right_steering_to_base_link" type="revolute">
-  <origin xyz="-0.10312 0.0505 0.0351" rpy="0 0 0"/>
+  <origin xyz="0.10312 -0.0505 0.0351" rpy="0 0 0"/>
   <parent link="base_link"/>
   <child link="right_steering_1"/>
@@ -153,5 +153,5 @@
 </joint>
 <joint name="left_steering_to_base_link" type="revolute">
-  <origin xyz="-0.10312 -0.0505 0.0351" rpy="0 0 0"/>
+  <origin xyz="0.10312 0.0505 0.0351" rpy="0 0 0"/>
   <parent link="base_link"/>
   <child link="left_steering_1"/>
@@ -160,17 +160,16 @@
 </joint>
 <joint name="left_rear_wheel_to_base_link" type="continuous">
-  <origin xyz="0.097623 -0.083 0.0351" rpy="0 0 0"/>
+  <origin xyz="-0.097623 0.083 0.0351" rpy="0 0 0"/>
   <parent link="base_link"/>
   <child link="left_rear_wheel_1"/>
-  <axis xyz="-0.0 -1.0 -0.0"/>
-</joint>
+  <axis xyz="0.0 1.0 0.0"/> </joint>
 <joint name="right_rear_wheel_to_base_link" type="continuous">
-  <origin xyz="0.098035 0.083 0.0351" rpy="0 0 0"/>
+  <origin xyz="-0.098035 -0.083 0.0351" rpy="0 0 0"/>
   <parent link="base_link"/>
   <child link="right_rear_wheel_1"/>
-  <axis xyz="0.0 -1.0 0.0"/>
+  <axis xyz="0.0 1.0 0.0"/>
 </joint>
 <joint name="right_front_wheel_to_right_steering" type="continuous">
-  <origin xyz="0.00307 0.032322 0.0" rpy="0 0 0"/>
+  <origin xyz="-0.00307 -0.032322 0.0" rpy="0 0 0"/>
   <parent link="right_steering_1"/>
   <child link="right_front_wheel_1"/>
@@ -178,8 +177,8 @@
 </joint>
 <joint name="left_front_wheel_to_left_steering" type="continuous">
-  <origin xyz="0.00307 -0.032322 0.0" rpy="0 0 0"/>
+  <origin xyz="-0.00307 0.032322 0.0" rpy="0 0 0"/>
   <parent link="left_steering_1"/>
   <child link="left_front_wheel_1"/>
-  <axis xyz="0.0 -1.0 -0.0"/>
+  <axis xyz="0.0 1.0 0.0"/>
 </joint>
 </robot>

Commit message: new map

File: robot_2_description/urdf/robot_2.xacro (robot description, xacro)
@@ -5,4 +5,6 @@
 <xacro:include filename="$(find robot_2_description)/urdf/robot_2.gazebo" />
 <xacro:include filename="$(find robot_2_description)/urdf/ros2_control.xacro" />
+<xacro:include filename="$(find robot_2_description)/urdf/lidar.xacro" />
+<xacro:include filename="$(find robot_2_description)/urdf/camera.xacro" />
 <link name="base_link">
   <inertial>
@@ -150,5 +152,5 @@
   <child link="right_steering_1"/>
   <axis xyz="0.0 0.0 1.0"/>
-  <limit lower="-0.6" upper="0.6" effort="100.0" velocity="10.0"/>
+  <limit lower="-0.785" upper="0.785" effort="100.0" velocity="10.0"/>
 </joint>
 <joint name="left_steering_to_base_link" type="revolute">
@@ -157,5 +159,5 @@
   <child link="left_steering_1"/>
   <axis xyz="0.0 0.0 1.0"/>
-  <limit lower="-0.6" upper="0.6" effort="100.0" velocity="10.0"/>
+  <limit lower="-0.785" upper="0.785" effort="100.0" velocity="10.0"/>
 </joint>
 <joint name="left_rear_wheel_to_base_link" type="continuous">

Commit message: do line

File: robot_2_description/urdf/robot_2.xacro (robot description, xacro)
@@ -152,5 +152,5 @@
   <child link="right_steering_1"/>
   <axis xyz="0.0 0.0 1.0"/>
-  <limit lower="-0.785" upper="0.785" effort="100.0" velocity="10.0"/>
+  <limit lower="-0.785" upper="0.785" effort="200.0" velocity="10.0"/>
 </joint>
 <joint name="left_steering_to_base_link" type="revolute">
@@ -159,5 +159,5 @@
   <child link="left_steering_1"/>
   <axis xyz="0.0 0.0 1.0"/>
-  <limit lower="-0.785" upper="0.785" effort="100.0" velocity="10.0"/>
+  <limit lower="-0.785" upper="0.785" effort="200.0" velocity="10.0"/>
 </joint>
 <joint name="left_rear_wheel_to_base_link" type="continuous">
