Commit message: fix file config

File: robot_2_description/urdf/robot_2.xacro (robot description, xacro)
@@ -152,5 +152,5 @@
   <child link="right_steering_1"/>
   <axis xyz="0.0 0.0 1.0"/>
-  <limit lower="-0.785" upper="0.785" effort="200.0" velocity="10.0"/>
+  <limit lower="-1.25" upper="1.25" effort="200.0" velocity="10.0"/>
 </joint>
 <joint name="left_steering_to_base_link" type="revolute">
@@ -159,5 +159,5 @@
   <child link="left_steering_1"/>
   <axis xyz="0.0 0.0 1.0"/>
-  <limit lower="-0.785" upper="0.785" effort="200.0" velocity="10.0"/>
+  <limit lower="-1.25" upper="1.25" effort="200.0" velocity="10.0"/>
 </joint>
 <joint name="left_rear_wheel_to_base_link" type="continuous">
